Commit message: Add LeArm URDF, meshes, launch files, and Gazebo configs

File: src/learm_ros2/packages/learm_ros2_description/urdf/gazebo.urdf.xacro (robot description, xacro)
@@ -48,14 +48,21 @@
             <inertia ixx="0.03" iyy="0.03" izz="0.03" ixy="0.0" ixz="0.0" iyz="0.0" />
         </inertial>
+        <collision>
+            <geometry>
+                <mesh filename="package://learm_ros2_description/meshes/forearm1.stl" scale="0.1 0.1 0.1"/>
+            </geometry>
+        </collision>
     </link>
     <link name="forearm1_link">
         <visual>
-            <geometry>
-                <mesh filename="package://learm_ros2_description/meshes/forearm1.stl" />
-            </geometry>
-        </visual>
-        <collision>
-            <geometry>
-                <mesh filename="package://learm_ros2_description/meshes/forearm1.stl" />
+            <origin rpy="0 0 3.14159"/>
+            <geometry>
+                <mesh filename="package://learm_ros2_description/meshes/forearm1.stl" scale="0.1 0.1 0.1"/>
+            </geometry>
+        </visual>
+        <collision>
+            <origin rpy="0 0 3.14159"/>
+            <geometry>
+                <mesh filename="package://learm_ros2_description/meshes/forearm1.stl" scale="0.1 0.1 0.1"/>
             </geometry>
         </collision>
@@ -66,21 +73,27 @@
     </link>
     <link name="forearm2_link">
-        <visual>
-            <geometry>
-                <mesh filename="package://learm_ros2_description/meshes/forearm2.stl" />
-            </geometry>
-        </visual>
-        <collision>
-            <geometry>
-                <mesh filename="package://learm_ros2_description/meshes/forearm2.stl" />
-            </geometry>
-        </collision>
-<inertial>
-            <mass value="0.1" />
-            <inertia ixx="0.03" iyy="0.03" izz="0.03" ixy="0.0" ixz="0.0" iyz="0.0" />
-        </inertial>
-    </link>
+  <visual>
+    <origin xyz="0 0 0" rpy="1.57 0 4.7"/>
+    <geometry>
+      <mesh filename="package://learm_ros2_description/meshes/forearm2.stl"
+            scale="0.1 0.1 0.1"/>
+    </geometry>
+  </visual>
+  <collision>
+    <origin xyz="0 0 0" rpy=" 1.57 0 4.7"/>
+    <geometry>
+      <mesh filename="package://learm_ros2_description/meshes/forearm2.stl"
+            scale="0.1 0.1 0.1"/>
+    </geometry>
+  </collision>
+  <inertial>
+    <mass value="0.1"/>
+    <inertia ixx="0.03" iyy="0.03" izz="0.03"
+             ixy="0.0" ixz="0.0" iyz="0.0"/>
+  </inertial>
+</link>
     <link name="wrist_link">
         <visual>
+            <origin rpy="0 0 3.14159"/>
             <geometry>
                 <mesh filename="package://learm_ros2_description/meshes/wrist.stl" />
@@ -88,4 +101,5 @@
         </visual>
         <collision>
+            <origin rpy="0 0 3.14159"/>
             <geometry>
                 <mesh filename="package://learm_ros2_description/meshes/wrist.stl" />
@@ -132,10 +146,10 @@
         <visual>
             <geometry>
-                <mesh filename="package://learm_ros2_description/meshes/carpal-left.stl" />
-            </geometry>
-        </visual>
-        <collision>
-            <geometry>
-                <mesh filename="package://learm_ros2_description/meshes/carpal-left.stl" />
+                <mesh filename="package://learm_ros2_description/meshes/carpal-right.stl" />
+            </geometry>
+        </visual>
+        <collision>
+            <geometry>
+                <mesh filename="package://learm_ros2_description/meshes/carpal-right.stl" />
             </geometry>
         </collision>
@@ -212,84 +226,84 @@
     </link>
     <joint name="shoulder_pan" type="revolute">
-        <parent link="base_link" />
-        <child link="shoulder_link" />
-        <origin xyz="0 0 0.059" />
-        <axis xyz="0 0 1" />
-        <limit lower="-1.57" upper="1.57" effort="1000" velocity="0.5" />
-    </joint>
+    <parent link="base_link"/>
+    <child link="shoulder_link"/>
+    <origin xyz="0 0 0.059"/>
+    <axis xyz="0 0 1"/>
+    <limit effort="1000" lower="-1.57" upper="1.57" velocity="0.5"/>
+  </joint>
     <joint name="shoulder_lift" type="revolute">
-        <parent link="shoulder_link" />
-        <child link="humerus_link" />
-        <origin xyz="-0.010 0 0.028" />
-        <axis xyz="0 1 0" />
-        <limit lower="-1.57" upper="1.57" effort="1000" velocity="0.5" />
-    </joint>
+    <parent link="shoulder_link"/>
+    <child link="humerus_link"/>
+    <origin xyz="-0.010 0 0.028"/>
+    <axis xyz="0 1 0"/>
+    <limit effort="1000" lower="-1.57" upper="1.57" velocity="0.5"/>
+  </joint>
     <joint name="elbow1" type="revolute">
-         <parent link="humerus_link"/>
-         <child link="forearm1_link"/>
-         <origin xyz="0 0 0.105"/>
-         <axis xyz="0 -1 0"/>
-         <limit effort="1000" lower="-1.57" upper="1.57" velocity="0.5"/>
-    </joint>
+    <parent link="humerus_link"/>
+    <child link="forearm1_link"/>
+    <origin xyz="0 0 0.105"/>
+    <axis xyz="0 -1 0"/>
+    <limit effort="1000" lower="-1.57" upper="1.57" velocity="0.5"/>
+  </joint>
     <joint name="elbow2" type="revolute">
-         <parent link="forearm1_link"/>
-         <child link="forearm2_link"/>
-         <origin xyz="0.0531 0 0.0186"/>
-         <axis xyz="0 0 -1"/>
-         <limit effort="1000" lower="-1.57" upper="1.57" velocity="0.5"/>
-    </joint>
-    <joint name="wrist_flex" type="revolute">
-        <parent link="forearm2_link" />
-        <child link="wrist_link" />
-        <origin xyz="0 0 0.090" />
-        <axis xyz="0 -1 0" />
-        <limit lower="-1.57" upper="1.57" effort="1000" velocity="0.5" />
-    </joint>
-    <joint name="wrist_roll" type="revolute">
-        <parent link="wrist_link" />
-        <child link="hand_link" />
-        <origin xyz="0 0 0.060" />
-        <axis xyz="0 0 1" />
-        <limit lower="-1.57" upper="1.57" effort="1000" velocity="0.5" />
-    </joint>
-    <joint name="grip_left" type="revolute">
-        <parent link="hand_link" />
-        <child link="grip_left_link" />
-        <origin xyz="0 +0.015 0.030" rpy="-1.57 0 0" />
-        <axis xyz="-1 0 0" />
-        <limit lower="-1.57" upper="0" effort="1000" velocity="0.5" />
-    </joint>
-    <joint name="grip_right" type="revolute">
-        <parent link="hand_link" />
-        <child link="grip_right_link" />
-        <origin xyz="0 -0.015 0.030" rpy="1.57 0 0" />
-        <axis xyz="-1 0 0" />
-        <limit lower="0" upper="1.57" effort="1000" velocity="0.5" />
-        <mimic joint="grip_left" multiplier="-1" />
-    </joint>
-    <joint name="tendon_left" type="revolute">
-        <parent link="hand_link" />
-        <child link="tendon_left_link" />
-        <origin xyz="0 +0.005 0.050" rpy="-1.57 0 0" />
-        <axis xyz="-1 0 0" />
-        <limit lower="-1.57" upper="0" effort="1000" velocity="0.5" />
-        <mimic joint="grip_left" />
-    </joint>
-    <joint name="tendon_right" type="revolute">
-        <parent link="hand_link" />
-        <child link="tendon_right_link" />
-        <origin xyz="0 -0.005 0.050" rpy="1.57 0 0" />
-        <axis xyz="-1 0 0" />
-        <limit lower="0" upper="1.57" effort="1000" velocity="0.5" />
-        <mimic joint="grip_left" multiplier="-1" />
-    </joint>
-    <joint name="finger_left" type="revolute">
-        <parent link="grip_left_link" />
-        <child link="finger_left_link" />
-        <origin xyz="0 0 0.030" rpy="1.57 0 0" />
-        <axis xyz="-1 0 0" />
-        <limit lower="-1.57" upper="0" effort="1000" velocity="0.5" />
-        <mimic joint="grip_left" multiplier="-1" />
-    </joint>
+    <parent link="forearm1_link"/>
+    <child link="forearm2_link"/>
+    <origin xyz="0.0531 0 0.0186"/>
+    <axis xyz="0 0 -1"/>
+    <limit effort="1000" lower="-1.57" upper="1.57" velocity="0.5"/>
+  </joint>
+  <joint name="wrist_flex" type="revolute">
+    <parent link="forearm2_link"/>
+    <child link="wrist_link"/>
+    <origin xyz="0 0 0.08"/>
+    <axis xyz="0 1 0"/>
+    <limit effort="1000" lower="-1.57" upper="1.57" velocity="0.5"/>
+  </joint>
+  <joint name="wrist_roll" type="revolute">
+    <parent link="wrist_link"/>
+    <child link="hand_link"/>
+    <origin xyz="0 0 0.060"/>
+    <axis xyz="0 0 1"/>
+    <limit effort="1000" lower="-1.57" upper="1.57" velocity="0.5"/>
+  </joint>
+   <joint name="grip_left" type="revolute">
+    <parent link="hand_link"/>
+    <child link="grip_left_link"/>
+    <origin rpy="-1.57 0 0" xyz="0 +0.015 0.030"/>
+    <axis xyz="-1 0 0"/>
+    <limit effort="1000" lower="-1.57" upper="0" velocity="0.5"/>
+  </joint>
+  <joint name="grip_right" type="revolute">
+    <parent link="hand_link"/>
+    <child link="grip_right_link"/>
+    <origin rpy="1.57 0 0" xyz="0 -0.015 0.030"/>
+    <axis xyz="-1 0 0"/>
+    <limit effort="1000" lower="0" upper="1.57" velocity="0.5"/>
+    <mimic joint="grip_left" multiplier="-1"/>
+  </joint>
+  <joint name="tendon_left" type="revolute">
+    <parent link="hand_link"/>
+    <child link="tendon_left_link"/>
+    <origin rpy="-1.57 0 0" xyz="0 +0.005 0.050"/>
+    <axis xyz="-1 0 0"/>
+    <limit effort="1000" lower="-1.57" upper="0" velocity="0.5"/>
+    <mimic joint="grip_left"/>
+  </joint>
+     <joint name="tendon_right" type="revolute">
+    <parent link="hand_link"/>
+    <child link="tendon_right_link"/>
+    <origin rpy="1.57 0 0" xyz="0 -0.005 0.050"/>
+    <axis xyz="-1 0 0"/>
+    <limit effort="1000" lower="0" upper="1.57" velocity="0.5"/>
+    <mimic joint="grip_left" multiplier="-1"/>
+  </joint>
+  <joint name="finger_left" type="revolute">
+    <parent link="grip_left_link"/>
+    <child link="finger_left_link"/>
+    <origin rpy="1.57 0 0" xyz="0 0 0.030"/>
+    <axis xyz="-1 0 0"/>
+    <limit effort="1000" lower="-1.57" upper="0" velocity="0.5"/>
+    <mimic joint="grip_left" multiplier="-1"/>
+  </joint>
     <joint name="finger_right" type="revolute">
         <parent link="grip_right_link" />
@@ -320,24 +334,24 @@
         </actuator>
     </transmission>
-    <transmission name="trans1_elbow">
+    <transmission name="trans_elbow">
         <type>transmission_interface/SimpleTransmission</type>
         <joint name="elbow1">
             <hardwareInterface>hardware_interface/EffortJointInterface</hardwareInterface>
         </joint>
-        <actuator name="elbow1_motor">
-            <hardwareInterface>hardware_interface/EffortJointInterface</hardwareInterface>
-            <mechanicalReduction>1</mechanicalReduction>
-        </actuator>
-    </transmission>
-    <transmission name="trans2_elbow">
-        <type>transmission_interface/SimpleTransmission</type>
-        <joint name="elbow2">
-            <hardwareInterface>hardware_interface/EffortJointInterface</hardwareInterface>
-        </joint>
-        <actuator name="elbow2_motor">
-            <hardwareInterface>hardware_interface/EffortJointInterface</hardwareInterface>
-            <mechanicalReduction>1</mechanicalReduction>
-        </actuator>
-    </transmission>
+        <actuator name="elbow_motor">
+            <hardwareInterface>hardware_interface/EffortJointInterface</hardwareInterface>
+            <mechanicalReduction>1</mechanicalReduction>
+        </actuator>
+    </transmission>
+    <transmission name="trans_forearm2">
+  <type>transmission_interface/SimpleTransmission</type>
+  <joint name="elbow2">
+    <hardwareInterface>hardware_interface/EffortJointInterface</hardwareInterface>
+  </joint>
+  <actuator name="forearm2_motor">
+    <hardwareInterface>hardware_interface/EffortJointInterface</hardwareInterface>
+    <mechanicalReduction>1</mechanicalReduction>
+  </actuator>
+</transmission>
     <transmission name="trans_wrist_flex">
         <type>transmission_interface/SimpleTransmission</type>

File: src/learm_ros2/packages/learm_ros2_description/urdf/learm.urdf.xacro (robot description, xacro)
@@ -8,5 +8,5 @@
     <visual>
       <geometry>
-        <mesh filename="package://learm_ros2_description/meshes/base.stl"/>
+        <mesh filename="package://learm_ros2_description/meshes/base.stl" />
       </geometry>
     </visual>
@@ -15,5 +15,5 @@
     <visual>
       <geometry>
-        <mesh filename="package://learm_ros2_description/meshes/shoulder.stl"/>
+        <mesh filename="package://learm_ros2_description/meshes/shoulder.stl" />
       </geometry>
     </visual>
@@ -22,5 +22,5 @@
     <visual>
       <geometry>
-        <mesh filename="package://learm_ros2_description/meshes/humerus.stl"/>
+        <mesh filename="package://learm_ros2_description/meshes/humerus.stl" />
       </geometry>
     </visual>
@@ -30,5 +30,5 @@
       <origin rpy="0 0 3.14159"/>
       <geometry>
-        <mesh filename="package://learm_ros2_description/meshes/forearm1.stl" scale="0.1 0.1 0.1"/>
+        <mesh filename="package://learm_ros2_description/meshes/forearm1.stl" scale="0.1 0.1 0.1" />
       </geometry>
     </visual>
@@ -46,5 +46,5 @@
       <origin rpy="0 0 3.14159"/>
       <geometry>
-        <mesh filename="package://learm_ros2_description/meshes/wrist.stl"/>
+        <mesh filename="package://learm_ros2_description/meshes/wrist.stl" />
       </geometry>
     </visual>
@@ -53,5 +53,5 @@
     <visual>
       <geometry>
-        <mesh filename="package://learm_ros2_description/meshes/hand.stl"/>
+        <mesh filename="package://learm_ros2_description/meshes/hand.stl" />
       </geometry>
     </visual>
@@ -60,5 +60,5 @@
     <visual>
       <geometry>
-        <mesh filename="package://learm_ros2_description/meshes/carpal-left.stl"/>
+        <mesh filename="package://learm_ros2_description/meshes/carpal-left.stl" />
       </geometry>
     </visual>
@@ -67,5 +67,5 @@
     <visual>
       <geometry>
-        <mesh filename="package://learm_ros2_description/meshes/carpal-right.stl"/>
+        <mesh filename="package://learm_ros2_description/meshes/carpal-right.stl" />
       </geometry>
     </visual>
@@ -74,5 +74,5 @@
     <visual>
       <geometry>
-        <mesh filename="package://learm_ros2_description/meshes/tendon.stl"/>
+        <mesh filename="package://learm_ros2_description/meshes/tendon.stl" />
       </geometry>
     </visual>
@@ -81,5 +81,5 @@
     <visual>
       <geometry>
-        <mesh filename="package://learm_ros2_description/meshes/tendon.stl"/>
+        <mesh filename="package://learm_ros2_description/meshes/tendon.stl" />
       </geometry>
     </visual>
@@ -88,5 +88,5 @@
     <visual>
       <geometry>
-        <mesh filename="package://learm_ros2_description/meshes/finger.stl"/>
+        <mesh filename="package://learm_ros2_description/meshes/finger.stl" />
       </geometry>
     </visual>
@@ -96,5 +96,5 @@
       <origin rpy="0 0 3.14159"/>
       <geometry>
-        <mesh filename="package://learm_ros2_description/meshes/finger.stl"/>
+        <mesh filename="package://learm_ros2_description/meshes/finger.stl" />
       </geometry>
     </visual>

Commit message: Initial commit from Ubuntu laptop

File: src/learm_ros2/packages/learm_ros2_description/urdf/gazebo.urdf.xacro (robot description, xacro)
@@ -1,4 +1,5 @@
 <?xml version="1.0" ?>
 <robot name="LeArm">
+    <link name="world"/>
     <link name="base_link">
         <visual>
@@ -225,4 +226,9 @@
         </inertial>
     </link>
+    <joint name="world_fixed_joint" type="fixed">
+  <parent link="world"/>
+  <child link="base_link"/>
+  <origin xyz="0 0 0" rpy="0 0 0"/>
+</joint>
     <joint name="shoulder_pan" type="revolute">
     <parent link="base_link"/>
@@ -434,8 +440,14 @@
         </actuator>
     </transmission>
-    <gazebo>
-        <plugin name="gazebo_ros_control" filename="libgazebo_ros_control.so">
-            <robotNamespace>/</robotNamespace>
-        </plugin>
-    </gazebo>
+<ros2_control name="LeArmSystem" type="system">
+  <hardware>
+    <!-- bridge into gazebo -->
+    <plugin>gazebo_ros2_control/GazeboSystem</plugin>
+  </hardware>
+</ros2_control>
+<gazebo>
+  <plugin name="gazebo_ros_control" filename="libgazebo_ros_control.so">
+    <robotNamespace>/</robotNamespace>
+  </plugin>
+</gazebo>
 </robot>
