Commit message: Fix Gazebo spawn and add FK node

File: src/learm_ros2/packages/learm_ros2_description/urdf/gazebo.urdf.xacro (robot description, xacro)
@@ -1,287 +1,137 @@
-<?xml version="1.0" ?>
-<robot name="LeArm">
-    <link name="world"/>
-    <link name="base_link">
-        <visual>
-            <geometry>
-                <mesh filename="package://learm_ros2_description/meshes/base.stl" />
-            </geometry>
-        </visual>
-        <collision>
-            <geometry>
-                <mesh filename="package://learm_ros2_description/meshes/base.stl" />
-            </geometry>
-        </collision>
-<inertial>
-            <mass value="0.1" />
-            <inertia ixx="0.03" iyy="0.03" izz="0.03" ixy="0.0" ixz="0.0" iyz="0.0" />
-        </inertial>
-    </link>
-    <link name="shoulder_link">
-        <visual>
-            <geometry>
-                <mesh filename="package://learm_ros2_description/meshes/shoulder.stl" />
-            </geometry>
-        </visual>
-        <collision>
-            <geometry>
-                <mesh filename="package://learm_ros2_description/meshes/shoulder.stl" />
-            </geometry>
-        </collision>
-<inertial>
-            <mass value="0.1" />
-            <inertia ixx="0.03" iyy="0.03" izz="0.03" ixy="0.0" ixz="0.0" iyz="0.0" />
-        </inertial>
-    </link>
-    <link name="humerus_link">
-        <visual>
-            <geometry>
-                <mesh filename="package://learm_ros2_description/meshes/humerus.stl" />
-            </geometry>
-        </visual>
-        <collision>
-            <geometry>
-                <mesh filename="package://learm_ros2_description/meshes/humerus.stl" />
-            </geometry>
-        </collision>
-<inertial>
-            <mass value="0.1" />
-            <inertia ixx="0.03" iyy="0.03" izz="0.03" ixy="0.0" ixz="0.0" iyz="0.0" />
-        </inertial>
-        <collision>
-            <geometry>
-                <mesh filename="package://learm_ros2_description/meshes/forearm1.stl" scale="0.1 0.1 0.1"/>
-            </geometry>
-        </collision>
-    </link>
-    <link name="forearm1_link">
-        <visual>
-            <origin rpy="0 0 3.14159"/>
-            <geometry>
-                <mesh filename="package://learm_ros2_description/meshes/forearm1.stl" scale="0.1 0.1 0.1"/>
-            </geometry>
-        </visual>
-        <collision>
-            <origin rpy="0 0 3.14159"/>
-            <geometry>
-                <mesh filename="package://learm_ros2_description/meshes/forearm1.stl" scale="0.1 0.1 0.1"/>
-            </geometry>
-        </collision>
-<inertial>
-            <mass value="0.1" />
-            <inertia ixx="0.03" iyy="0.03" izz="0.03" ixy="0.0" ixz="0.0" iyz="0.0" />
-        </inertial>
-    </link>
-    <link name="forearm2_link">
-  <visual>
-    <origin xyz="0 0 0" rpy="1.57 0 4.7"/>
-    <geometry>
-      <mesh filename="package://learm_ros2_description/meshes/forearm2.stl"
-            scale="0.1 0.1 0.1"/>
-    </geometry>
-  </visual>
-  <collision>
-    <origin xyz="0 0 0" rpy=" 1.57 0 4.7"/>
-    <geometry>
-      <mesh filename="package://learm_ros2_description/meshes/forearm2.stl"
-            scale="0.1 0.1 0.1"/>
-    </geometry>
-  </collision>
-  <inertial>
-    <mass value="0.1"/>
-    <inertia ixx="0.03" iyy="0.03" izz="0.03"
-             ixy="0.0" ixz="0.0" iyz="0.0"/>
-  </inertial>
-</link>
-    <link name="wrist_link">
-        <visual>
-            <origin rpy="0 0 3.14159"/>
-            <geometry>
-                <mesh filename="package://learm_ros2_description/meshes/wrist.stl" />
-            </geometry>
-        </visual>
-        <collision>
-            <origin rpy="0 0 3.14159"/>
-            <geometry>
-                <mesh filename="package://learm_ros2_description/meshes/wrist.stl" />
-            </geometry>
-        </collision>
-<inertial>
-            <mass value="0.1" />
-            <inertia ixx="0.03" iyy="0.03" izz="0.03" ixy="0.0" ixz="0.0" iyz="0.0" />
-        </inertial>
-    </link>
-    <link name="hand_link">
-        <visual>
-            <geometry>
-                <mesh filename="package://learm_ros2_description/meshes/hand.stl" />
-            </geometry>
-        </visual>
-        <collision>
-            <geometry>
-                <mesh filename="package://learm_ros2_description/meshes/hand.stl" />
-            </geometry>
-        </collision>
-<inertial>
-            <mass value="0.1" />
-            <inertia ixx="0.03" iyy="0.03" izz="0.03" ixy="0.0" ixz="0.0" iyz="0.0" />
-        </inertial>
-    </link>
-    <link name="grip_left_link">
-        <visual>
-            <geometry>
-                <mesh filename="package://learm_ros2_description/meshes/carpal-left.stl" />
-            </geometry>
-        </visual>
-        <collision>
-            <geometry>
-                <mesh filename="package://learm_ros2_description/meshes/carpal-left.stl" />
-            </geometry>
-        </collision>
-<inertial>
-            <mass value="0.1" />
-            <inertia ixx="0.03" iyy="0.03" izz="0.03" ixy="0.0" ixz="0.0" iyz="0.0" />
-        </inertial>
-    </link>
-    <link name="grip_right_link">
-        <visual>
-            <geometry>
-                <mesh filename="package://learm_ros2_description/meshes/carpal-right.stl" />
-            </geometry>
-        </visual>
-        <collision>
-            <geometry>
-                <mesh filename="package://learm_ros2_description/meshes/carpal-right.stl" />
-            </geometry>
-        </collision>
-<inertial>
-            <mass value="0.1" />
-            <inertia ixx="0.03" iyy="0.03" izz="0.03" ixy="0.0" ixz="0.0" iyz="0.0" />
-        </inertial>
-    </link>
-    <link name="tendon_left_link">
-        <visual>
-            <geometry>
-                <mesh filename="package://learm_ros2_description/meshes/tendon.stl" />
-            </geometry>
-        </visual>
-        <collision>
-            <geometry>
-                <mesh filename="package://learm_ros2_description/meshes/tendon.stl" />
-            </geometry>
-        </collision>
-<inertial>
-            <mass value="0.1" />
-            <inertia ixx="0.03" iyy="0.03" izz="0.03" ixy="0.0" ixz="0.0" iyz="0.0" />
-        </inertial>
-    </link>
-    <link name="tendon_right_link">
-        <visual>
-            <geometry>
-                <mesh filename="package://learm_ros2_description/meshes/tendon.stl" />
-            </geometry>
-        </visual>
-        <collision>
-            <geometry>
-                <mesh filename="package://learm_ros2_description/meshes/tendon.stl" />
-            </geometry>
-        </collision>
-<inertial>
-            <mass value="0.1" />
-            <inertia ixx="0.03" iyy="0.03" izz="0.03" ixy="0.0" ixz="0.0" iyz="0.0" />
-        </inertial>
-    </link>
-    <link name="finger_left_link">
-        <visual>
-            <geometry>
-                <mesh filename="package://learm_ros2_description/meshes/finger.stl" />
-            </geometry>
-        </visual>
-        <collision>
-            <geometry>
-                <mesh filename="package://learm_ros2_description/meshes/finger.stl" />
-            </geometry>
-        </collision>
-<inertial>
-            <mass value="0.1" />
-            <inertia ixx="0.03" iyy="0.03" izz="0.03" ixy="0.0" ixz="0.0" iyz="0.0" />
-        </inertial>
-    </link>
-    <link name="finger_right_link">
-        <visual>
-            <origin rpy="0 0 3.14159" />
-            <geometry>
-                <mesh filename="package://learm_ros2_description/meshes/finger.stl" />
-            </geometry>
-        </visual>
-        <collision>
-            <origin rpy="0 0 3.14159" />
-            <geometry>
-                <mesh filename="package://learm_ros2_description/meshes/finger.stl" />
-            </geometry>
-        </collision>
-<inertial>
-            <mass value="0.1" />
-            <inertia ixx="0.03" iyy="0.03" izz="0.03" ixy="0.0" ixz="0.0" iyz="0.0" />
-        </inertial>
-    </link>
-    <joint name="world_fixed_joint" type="fixed">
-  <parent link="world"/>
-  <child link="base_link"/>
-  <origin xyz="0 0 0" rpy="0 0 0"/>
-</joint>
-    <joint name="shoulder_pan" type="revolute">
-    <parent link="base_link"/>
-    <child link="shoulder_link"/>
-    <origin xyz="0 0 0.059"/>
+<?xml version="1.0"?>
+<robot name="LeArm" xmlns:xacro="http://www.ros.org/wiki/xacro">
+  <!-- args passed from launch -->
+  <xacro:arg name="mesh_dir" default=""/>
+  <xacro:arg name="ros2_control_params" default=""/>
+  <!-- bind args to xacro properties -->
+  <xacro:property name="mesh_root" value="$(arg mesh_dir)"/>
+  <xacro:property name="ctrl_yaml"  value="$(arg ros2_control_params)"/>
+  <!-- Gazebo Classic loads meshes most reliably via file:// -->
+  <xacro:property name="MESH" value="file://${mesh_root}/meshes"/>
+  <!-- ===== LINKS ===== -->
+  <link name="world"/>
+  <link name="base_link">
+    <visual><geometry><mesh filename="${MESH}/base.stl"/></geometry></visual>
+    <collision><geometry><mesh filename="${MESH}/base.stl"/></geometry></collision>
+    <inertial><mass value="0.1"/><inertia ixx="0.03" iyy="0.03" izz="0.03" ixy="0" ixz="0" iyz="0"/></inertial>
+  </link>
+  <link name="shoulder_link">
+    <visual><geometry><mesh filename="${MESH}/shoulder.stl"/></geometry></visual>
+    <collision><geometry><mesh filename="${MESH}/shoulder.stl"/></geometry></collision>
+    <inertial><mass value="0.1"/><inertia ixx="0.03" iyy="0.03" izz="0.03" ixy="0" ixz="0" iyz="0"/></inertial>
+  </link>
+  <link name="humerus_link">
+    <visual><geometry><mesh filename="${MESH}/humerus.stl"/></geometry></visual>
+    <collision><geometry><mesh filename="${MESH}/humerus.stl"/></geometry></collision>
+    <inertial><mass value="0.1"/><inertia ixx="0.03" iyy="0.03" izz="0.03" ixy="0" ixz="0" iyz="0"/></inertial>
+  </link>
+  <link name="forearm1_link">
+    <visual><origin rpy="0 0 3.14159"/><geometry><mesh filename="${MESH}/forearm1.stl" scale="0.1 0.1 0.1"/></geometry></visual>
+    <collision><origin rpy="0 0 3.14159"/><geometry><mesh filename="${MESH}/forearm1.stl" scale="0.1 0.1 0.1"/></geometry></collision>
+    <inertial><mass value="0.1"/><inertia ixx="0.03" iyy="0.03" izz="0.03" ixy="0" ixz="0" iyz="0"/></inertial>
+  </link>
+  <link name="forearm2_link">
+    <visual><origin xyz="0 0 0" rpy="1.57 0 4.7"/><geometry><mesh filename="${MESH}/forearm2.stl" scale="0.1 0.1 0.1"/></geometry></visual>
+    <collision><origin xyz="0 0 0" rpy="1.57 0 4.7"/><geometry><mesh filename="${MESH}/forearm2.stl" scale="0.1 0.1 0.1"/></geometry></collision>
+    <inertial><mass value="0.1"/><inertia ixx="0.03" iyy="0.03" izz="0.03" ixy="0" ixz="0" iyz="0"/></inertial>
+  </link>
+  <link name="wrist_link">
+    <visual><origin rpy="0 0 3.14159"/><geometry><mesh filename="${MESH}/wrist.stl"/></geometry></visual>
+    <collision><origin rpy="0 0 3.14159"/><geometry><mesh filename="${MESH}/wrist.stl"/></geometry></collision>
+    <inertial><mass value="0.1"/><inertia ixx="0.03" iyy="0.03" izz="0.03" ixy="0" ixz="0" iyz="0"/></inertial>
+  </link>
+  <link name="hand_link">
+    <visual><geometry><mesh filename="${MESH}/hand.stl"/></geometry></visual>
+    <collision><geometry><mesh filename="${MESH}/hand.stl"/></geometry></collision>
+    <inertial><mass value="0.1"/><inertia ixx="0.03" iyy="0.03" izz="0.03" ixy="0" ixz="0" iyz="0"/></inertial>
+  </link>
+  <link name="grip_left_link">
+    <visual><geometry><mesh filename="${MESH}/carpal-left.stl"/></geometry></visual>
+    <collision><geometry><mesh filename="${MESH}/carpal-left.stl"/></geometry></collision>
+    <inertial><mass value="0.1"/><inertia ixx="0.03" iyy="0.03" izz="0.03" ixy="0" ixz="0" iyz="0"/></inertial>
+  </link>
+  <link name="grip_right_link">
+    <visual><geometry><mesh filename="${MESH}/carpal-right.stl"/></geometry></visual>
+    <collision><geometry><mesh filename="${MESH}/carpal-right.stl"/></geometry></collision>
+    <inertial><mass value="0.1"/><inertia ixx="0.03" iyy="0.03" izz="0.03" ixy="0" ixz="0" iyz="0"/></inertial>
+  </link>
+  <link name="tendon_left_link">
+    <visual><geometry><mesh filename="${MESH}/tendon.stl"/></geometry></visual>
+    <collision><geometry><mesh filename="${MESH}/tendon.stl"/></geometry></collision>
+    <inertial><mass value="0.1"/><inertia ixx="0.03" iyy="0.03" izz="0.03" ixy="0" ixz="0" iyz="0"/></inertial>
+  </link>
+  <link name="tendon_right_link">
+    <visual><geometry><mesh filename="${MESH}/tendon.stl"/></geometry></visual>
+    <collision><geometry><mesh filename="${MESH}/tendon.stl"/></geometry></collision>
+    <inertial><mass value="0.1"/><inertia ixx="0.03" iyy="0.03" izz="0.03" ixy="0" ixz="0" iyz="0"/></inertial>
+  </link>
+  <link name="finger_left_link">
+    <visual><geometry><mesh filename="${MESH}/finger.stl"/></geometry></visual>
+    <collision><geometry><mesh filename="${MESH}/finger.stl"/></geometry></collision>
+    <inertial><mass value="0.1"/><inertia ixx="0.03" iyy="0.03" izz="0.03" ixy="0" ixz="0" iyz="0"/></inertial>
+  </link>
+  <link name="finger_right_link">
+    <visual><origin rpy="0 0 3.14159"/><geometry><mesh filename="${MESH}/finger.stl"/></geometry></visual>
+    <collision><origin rpy="0 0 3.14159"/><geometry><mesh filename="${MESH}/finger.stl"/></geometry></collision>
+    <inertial><mass value="0.1"/><inertia ixx="0.03" iyy="0.03" izz="0.03" ixy="0" ixz="0" iyz="0"/></inertial>
+  </link>
+  <!-- ===== JOINTS ===== -->
+  <joint name="world_fixed_joint" type="fixed">
+    <parent link="world"/>
+    <child link="base_link"/>
+    <origin xyz="0 0 0" rpy="0 0 0"/>
+  </joint>
+  <joint name="shoulder_pan" type="revolute">
+    <parent link="base_link"/><child link="shoulder_link"/>
+    <origin xyz="0 0 0.059" rpy="0 0 0"/>
     <axis xyz="0 0 1"/>
     <limit effort="1000" lower="-1.57" upper="1.57" velocity="0.5"/>
-  </joint>
-    <joint name="shoulder_lift" type="revolute">
-    <parent link="shoulder_link"/>
-    <child link="humerus_link"/>
-    <origin xyz="-0.010 0 0.028"/>
+    <dynamics damping="2.0" friction="0.5"/>
+  </joint>
+  <joint name="shoulder_lift" type="revolute">
+    <parent link="shoulder_link"/><child link="humerus_link"/>
+    <origin xyz="-0.010 0 0.028" rpy="0 0 0"/>
     <axis xyz="0 1 0"/>
     <limit effort="1000" lower="-1.57" upper="1.57" velocity="0.5"/>
-  </joint>
-    <joint name="elbow1" type="revolute">
-    <parent link="humerus_link"/>
-    <child link="forearm1_link"/>
-    <origin xyz="0 0 0.105"/>
+    <dynamics damping="2.0" friction="0.5"/>
+  </joint>
+  <joint name="elbow1" type="revolute">
+    <parent link="humerus_link"/><child link="forearm1_link"/>
+    <origin xyz="0 0 0.105" rpy="0 0 0"/>
     <axis xyz="0 -1 0"/>
     <limit effort="1000" lower="-1.57" upper="1.57" velocity="0.5"/>
-  </joint>
-    <joint name="elbow2" type="revolute">
-    <parent link="forearm1_link"/>
-    <child link="forearm2_link"/>
-    <origin xyz="0.0531 0 0.0186"/>
+    <dynamics damping="2.0" friction="0.5"/>
+  </joint>
+  <joint name="elbow2" type="revolute">
+    <parent link="forearm1_link"/><child link="forearm2_link"/>
+    <origin xyz="0.0531 0 0.0186" rpy="0 0 0"/>
     <axis xyz="0 0 -1"/>
     <limit effort="1000" lower="-1.57" upper="1.57" velocity="0.5"/>
+    <dynamics damping="2.0" friction="0.5"/>
   </joint>
   <joint name="wrist_flex" type="revolute">
-    <parent link="forearm2_link"/>
-    <child link="wrist_link"/>
-    <origin xyz="0 0 0.08"/>
+    <parent link="forearm2_link"/><child link="wrist_link"/>
+    <origin xyz="0 0 0.08" rpy="0 0 0"/>
     <axis xyz="0 1 0"/>
     <limit effort="1000" lower="-1.57" upper="1.57" velocity="0.5"/>
+    <dynamics damping="1.5" friction="0.4"/>
   </joint>
   <joint name="wrist_roll" type="revolute">
-    <parent link="wrist_link"/>
-    <child link="hand_link"/>
-    <origin xyz="0 0 0.060"/>
+    <parent link="wrist_link"/><child link="hand_link"/>
+    <origin xyz="0 0 0.060" rpy="0 0 0"/>
     <axis xyz="0 0 1"/>
     <limit effort="1000" lower="-1.57" upper="1.57" velocity="0.5"/>
-  </joint>
-   <joint name="grip_left" type="revolute">
-    <parent link="hand_link"/>
-    <child link="grip_left_link"/>
-    <origin rpy="-1.57 0 0" xyz="0 +0.015 0.030"/>
+    <dynamics damping="1.5" friction="0.4"/>
+  </joint>
+  <!-- gripper joints left as-is (they can droop unless controlled) -->
+  <joint name="grip_left" type="revolute">
+    <parent link="hand_link"/><child link="grip_left_link"/>
+    <origin xyz="0 0.015 0.030" rpy="-1.57 0 0"/>
     <axis xyz="-1 0 0"/>
     <limit effort="1000" lower="-1.57" upper="0" velocity="0.5"/>
   </joint>
   <joint name="grip_right" type="revolute">
-    <parent link="hand_link"/>
-    <child link="grip_right_link"/>
-    <origin rpy="1.57 0 0" xyz="0 -0.015 0.030"/>
+    <parent link="hand_link"/><child link="grip_right_link"/>
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
File: src/learm_ros2/packages/learm_ros2_description/urdf/learm.urdf.xacro (robot description, xacro)
@@ -2,5 +2,5 @@
 <!-- =================================================================================== -->
 <!-- |    This document was autogenerated by xacro from src/learm_ros2/urdf/learm.urdf | -->
-<!-- |    EDITING THIS FILE BY HAND IS NOT RECOMMENDED                                 | -->
+<!-- |    EDITING THIS FILE BY HAND IS NOT RECOMMENDED          <mesh filename="package://learm_ros2_description/meshes/base.stl" />                       | -->
 <!-- =================================================================================== -->
 <robot name="learm">
@@ -8,5 +8,5 @@
     <visual>
       <geometry>
-        <mesh filename="package://learm_ros2_description/meshes/base.stl" />
+      <mesh filename="file:///home/skhizar/learm_ws/install/learm_ros2_description/share/learm_ros2_description/meshes/base.stl"/>
       </geometry>
     </visual>
